Commit message: peg-in-hole simulation updated, PID controllers for gravity compensation updated

File: sawyer_sim_examples/models/peg_hole/hole_0001.urdf (robot description, URDF)
Before this commit: robot hole_0001, 1 links, 0 joints
Links:
- added link world
Joints:
- added joint base_joint: type fixed, parent world, child hole_0001, origin xyz=0 0 0 rpy=0 0 0
