Commit message: peg-in-hole demo added to sawyer_sim_examples

File: sawyer_sim_examples/models/peg_hole/peg_0001.urdf (robot description, URDF)
Before this commit: robot peg_0001, 1 links, 0 joints
Links:
- link peg_0001: mass 0.193 -> 0.050

Commit message: Collision areas for peg-in-hole demo modified to reduce computational cost, positions and velocitires reduced

File: sawyer_sim_examples/models/peg_hole/peg_0001.urdf (robot description, URDF)
Before this commit: robot peg_0001, 1 links, 0 joints
Links:
- link peg_0001: geometry collision cylinder length=0.170 radius=0.02; visual mesh filename=package://sawyer_sim_examples/models/peg_hole/STL/rigid_peg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 scale=0.001 0.001 0.001

Commit message: controllers gain updated, peg-in-hole demo updated to work with SawyerRobot class, and frictions in hole decresased to facilitate the insertion, obtain data with movement sequence can be used with /robot/ati_ft_sensor_topic/ for real ATI sensor

File: sawyer_sim_examples/models/peg_hole/peg_0001.urdf (robot description, URDF)
Before this commit: robot peg_0001, 1 links, 0 joints
Links:
- link peg_0001: mass 0.050 -> 0.193
